File: christmas_light_controller.sch (KiCad schematic (older format))
At the start: 15 parts

Commit message: (wip) began relay_output schematic
Parts:
- added NT?: Net-Tie_4, symbol Device:Net-Tie_4
Connections:
- net 24V_GND: now also NT?.1
- net 3.3V_GND: now also NT?.2; no longer C?.2, R?.2
- net RELAY_1_EN: now reaches U?.24 (PA15)
- net A_GND: now reaches U?.5 (GNDANA)
- net A_GND: now also C?.2, R?.2, NT?.4
- new net PE: NT?.3
Changed lines of the file:
@@
 $Descr A4 11693 8268
 encoding utf-8
-Sheet 1 3
+Sheet 1 4
 Title ""
 Date ""
@@
 Comment4 ""
 $EndDescr
-$Sheet
-S 950  2000 550  700
-U 608C0A2A
-F0 "power_supply_3.3VDC" 50
-F1 "power_supply_3.3VDC.sch" 50
-F2 "+24V" I R 1500 2100 50
-F3 "GND" I R 1500 2250 50
-F4 "+3.3V" O R 1500 2400 50
-F5 "3.3V_GND" O R 1500 2550 50
-$EndSheet
 Text HLabel 1550 1000 2    50   UnSpc ~ 0
 +24V
@@
 F2 "+24V" O R 1500 1000 50
 F3 "24V_GND" O R 1500 1150 50
+F4 "PE" O R 1500 1300 50
 $EndSheet
 Text HLabel 1550 2100 2    50   UnSpc ~ 0
 +24V
-Text HLabel 1550 2250 2    50   UnSpc ~ 0
-GND
 Wire Wire Line
 	1500 2100 1550 2100
-Wire Wire Line
-	1550 2250 1500 2250
 $Comp
 L my_kicad_sch_lib:ATSAMD20G16B U?
@@
 Wire Wire Line
 	8650 3650 8600 3650
-Text HLabel 6200 3450 3    50   UnSpc ~ 0
-3.3V_GND
 Text HLabel 7350 4150 0    50   UnSpc ~ 0
 3.3V_GND
@@
 Wire Wire Line
 	6650 2650 6650 2700
-Text HLabel 6650 3050 3    50   UnSpc ~ 0
-3.3V_GND
 Wire Wire Line
 	6650 3000 6650 3050
@@
 Wire Wire Line
 	6200 3450 6200 3400
+$Sheet
+S 950  3050 550  700
+U 609B6707
+F0 "relay_output" 50
+F1 "relay_output.sch" 50
+F2 "+24V" I R 1500 3150 50
+F3 "RELAY_1_EN" I R 1500 3600 50
+F4 "24V_GND" I R 1500 3300 50
+$EndSheet
+Text HLabel 1550 3150 2    50   UnSpc ~ 0
++24V
+Wire Wire Line
+	1500 3150 1550 3150
+Text HLabel 1550 3600 2    50   UnSpc ~ 0
+RELAY_1_EN
+Text HLabel 7350 4750 0    50   UnSpc ~ 0
+RELAY_1_EN
+Wire Wire Line
+	7350 4750 7400 4750
+Wire Wire Line
+	1500 3600 1550 3600
+$Sheet
+S 950  2000 550  700
+U 608C0A2A
+F0 "power_supply_3.3VDC" 50
+F1 "power_supply_3.3VDC.sch" 50
+F2 "+24V" I R 1500 2100 50
+F3 "+3.3V" O R 1500 2400 50
+F4 "3.3V_GND" O R 1500 2550 50
+$EndSheet
+Text HLabel 3600 950  2    50   UnSpc ~ 0
+3.3V_GND
+Text HLabel 3300 950  0    50   UnSpc ~ 0
+24V_GND
+Wire Wire Line
+	3300 950  3350 950
+Wire Wire Line
+	3350 1050 3300 1050
+Text HLabel 7350 2850 0    50   UnSpc ~ 0
+A_GND
+Wire Wire Line
+	7400 2850 7350 2850
+Text HLabel 6650 3050 3    50   UnSpc ~ 0
+A_GND
+Text HLabel 6200 3450 3    50   UnSpc ~ 0
+A_GND
+Text HLabel 3600 1050 2    50   UnSpc ~ 0
+A_GND
+Wire Wire Line
+	3550 1050 3600 1050
+Text HLabel 1550 3300 2    50   UnSpc ~ 0
+24V_GND
+Wire Wire Line
+	1550 3300 1500 3300
+$Comp
+L Device:Net-Tie_4 NT?
+U 1 1 609C68A7
+P 3450 950
+F 0 "NT?" H 3450 1131 50  0000 C CNN
+F 1 "Net-Tie_4" H 3450 1040 50  0000 C CNN
+F 2 "" H 3450 950 50  0001 C CNN
+F 3 "~" H 3450 950 50  0001 C CNN
+	1    3450 950
+	1    0    0    -1
+$EndComp
+Wire Wire Line
+	3550 950  3600 950
+Text HLabel 3300 1050 0    50   UnSpc ~ 0
+PE
+Text HLabel 1550 1300 2    50   UnSpc ~ 0
+PE
+Wire Wire Line
+	1550 1300 1500 1300
 $EndSCHEMATC
